File: pcb/psu.sch (KiCad schematic (older format))
At the start: 6 parts, among them J7 Barrel_Jack_Switch, J8 30V input, J9 5V input bypass, U4 LM78M05_TO252

Commit message: layout check in
Parts:
- C26, C27: footprint Capacitor_SMD:C_0603_1608Metric -> Capacitor_SMD:C_0402_1005Metric
Changed lines of the file:
@@
 F 0 "C26" H 2915 1946 50  0000 L CNN
 F 1 "1u" H 2915 1855 50  0000 L CNN
-F 2 "Capacitor_SMD:C_0603_1608Metric" H 2838 1750 50  0001 C CNN
+F 2 "Capacitor_SMD:C_0402_1005Metric" H 2838 1750 50  0001 C CNN
 F 3 "~" H 2800 1900 50  0001 C CNN
 	1    2800 1900
@@
 F 0 "C27" H 4915 1946 50  0000 L CNN
 F 1 "1u" H 4915 1855 50  0000 L CNN
-F 2 "Capacitor_SMD:C_0603_1608Metric" H 4838 1750 50  0001 C CNN
+F 2 "Capacitor_SMD:C_0402_1005Metric" H 4838 1750 50  0001 C CNN
 F 3 "~" H 4800 1900 50  0001 C CNN
 	1    4800 1900
