File: pcb/vga.sch (KiCad schematic (older format))
At the start: 23 parts, among them J2 Input, J3 Output, U1 HMC625B

Commit message: final tweaks and produce outputs for jlcpcb fabrication
Parts:
- FB1, FB2: footprint Inductor_SMD:L_0603_1608Metric -> Inductor_SMD:L_0805_2012Metric
- R1: footprint Resistor_SMD:R_0402_1005Metric -> Resistor_SMD:R_0805_2012Metric_Pad1.20x1.40mm_HandSolder
Changed lines of the file:
@@
 F 0 "R1" V 7743 1700 50  0000 C CNN
 F 1 "1.8" V 7834 1700 50  0000 C CNN
-F 2 "Resistor_SMD:R_0402_1005Metric" V 7880 1700 50  0000 C CNN
+F 2 "Resistor_SMD:R_0805_2012Metric_Pad1.20x1.40mm_HandSolder" V 7880 1700 50  0000 C CNN
 F 3 "~" H 7950 1700 50  0001 C CNN
 	1    7950 1700
@@
 F 0 "FB2" V 7326 1700 50  0000 C CNN
 F 1 "GZ2012D601TF" V 7417 1700 50  0000 C CNN
-F 2 "Inductor_SMD:L_0603_1608Metric" V 7530 1700 50  0001 C CNN
+F 2 "Inductor_SMD:L_0805_2012Metric" V 7530 1700 50  0001 C CNN
 F 3 "~" H 7600 1700 50  0001 C CNN
 	1    7600 1700
@@
 F 0 "FB1" V 4576 1600 50  0000 C CNN
 F 1 "GZ2012D601TF" V 4667 1600 50  0000 C CNN
-F 2 "Inductor_SMD:L_0603_1608Metric" V 4780 1600 50  0001 C CNN
+F 2 "Inductor_SMD:L_0805_2012Metric" V 4780 1600 50  0001 C CNN
 F 3 "~" H 4850 1600 50  0001 C CNN
 	1    4850 1600
